File: small/siren_chorus/siren.sch (EAGLE design)
At the start: 50 parts, among them IC1 NE5532, IC2 PT2399, Q1 2N5457

Commit message: formatting updates
Parts:
- C1: value 100uF -> 100u
- C10, C11, C16, C17, C2, C9: value 0.1uF -> 100n
- C12: value 0.1uF -> 3n3
- C13: value 0.1uF -> 10n
- C14: value 10nF -> 100n
- C15: value 3.3nF -> 100n
- C3: value 0.01uF -> 10n
- C4: value 47uF -> 47u
- C5: value 10uF -> 47u
- C6: value 47uF -> 10u
- C7: value 10uF -> 10u
- C8: value 3.9nF -> 3n9
- R1: value 220k -> 1M
- R3: value 1M -> 220k
- RATE: value 100k -> 100kB
Connections:
- removed net N$27: C3.1, IC1_A.OUT, R5.1, R9.2
- new net N$30: C3.1, IC1_A.OUT, R6.1, R9.2
- net +9V: now also PAD2.P$1; no longer PAD1.P$1
- net GND: now also R10.1; no longer R11.1
- net IN: now also PAD1.P$1, R1.2; no longer PAD2.P$1, R3.2
- net N$1: now also C12.1; no longer C15.1
- net N$10: now also C15.1; no longer C12.1
- net N$11: now also C15.2; no longer C12.2
- net N$14: now also R11.1; no longer R10.1
- net N$15: now also R11.2; no longer R10.2
- net N$18: now also C5.+; no longer C6.+
- net N$2: now also C12.2; no longer C15.2
- net N$23: now also C9.1; no longer C10.1
- net N$24: now also C10.1; no longer C9.1
- net N$25: now also R3.2, R6.2; no longer R1.2, R5.2
- net N$26: now also R5.2; no longer R6.2
- net N$28: now also C6.+, R5.1; no longer C5.+, R6.1
- net N$31: now also R10.2; no longer R11.2
- net N$5: now also C13.1, R18.2; no longer C14.1, R20.2
- net N$6: now also C14.1, R20.2; no longer C13.1, R18.2
- net N$7: now also C13.2; no longer C14.2
- net N$9: now also C14.2; no longer C13.2
Other:
- moved on the sheet: C10, C12, C13, C14, C15, C16, C2, C3, C5, C6, C9, IC1_A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
