File: small/cyclops_fuzz/cyclops.brd (EAGLE design)
At the start: 33 x 52.1 mm, 44 parts, among them IC1 4558, IC2 741

Commit message: add EAGLE library, update 1590a chorus and tremolo, other minor edits
Parts:
- C2: value 200uF -> 100u
Changed lines of the file:
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@@
 <elements>
 <element name="C1" library="capacitors-film" package="BOX_SMALL" value="150nF" x="12.7" y="2.54" rot="R180"/>
-<element name="C2" library="capacitors-elec" package="063_025" value="200uF" x="3.81" y="3.81"/>
+<element name="C2" library="capacitors-elec" package="063_025" value="100u" x="3.81" y="3.81"/>
 <element name="C3" library="capacitors-film" package="BOX_MED" value="1uF" x="3.81" y="12.7" rot="R270"/>
 <element name="C6" library="capacitors-film" package="BOX_SMALL" value=".22uF" x="10.16" y="27.94" rot="R270"/>
