File: 1590a/janus_overdrive/janus.brd (EAGLE design)
At the start: 33 x 33.7 mm, 28 parts, among them IC1 LM741

Commit message: finished chorus and tremolo baords; other tweaks & polish
Parts:
- removed PAD1, PAD2, PAD5: PADSQR, supply pins:SQUARE
- removed PAD3, PAD4: PADRND, supply pins:ROUND
- added 9V: DC_MONO, jacks:DC
- added GND: PADRND, supply pins:ROUND
- added IN, OUT: PADSQR, supply pins:SQUARE
- C1, C3, C5: device capacitors-film:BOX_SMALL -> capacitors-film:050X030_025_2
- D1: device diodes:DO41-2 -> diodes:DO41-3
- moved D1 0.64 mm to (7.62, 22.9)
- moved C5 0.63 mm to (5.08, 24.1)
- moved R4 0.63 mm to (2.54, 22.9)
Connections:
- removed net +9V: D1.A, PAD1.1
- new net N$11: 9V.T, D1.A
- net GND: now also 9V.S, GND.1; no longer PAD3.1, PAD4.1
- net IN: now also IN.1; no longer PAD2.1
- net OUT: now also OUT.1; no longer PAD5.1
Routing:
- net +9V: track 4.49 -> 0.00 mm
- net N$11: track 0.00 -> 4.49 mm
- net N$12: track 20.3 -> 18.4 mm
- net N$3: track 17.2 -> 17.9 mm
- net N$10: track 3.81 -> 3.17 mm
- net CLIP: track 14.5 -> 14.0 mm
Other:
- board size 33 x 33.7 mm -> 33 x 33 mm
- board text added: "(c)2016"
- board text added: "JANUS"
- board text added: "OVERDRIVE/DIST"
- board text added: "burr settles"
- board text removed: "(c) 2016 burr settles"
- board text removed: "+9V"
- board text removed: "GND"
- board text removed: "IN"
- board text removed: "JANUS DRIVE"
- board text removed: "OUT"

Commit message: little edits & cleanup
Other:
- board text added: "OD+DISTORTION"
- board text removed: "OVERDRIVE/DIST"
Changed lines of the file:
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@@
 <text x="22.86" y="1.27" size="0.8128" layer="25" font="vector">burr settles</text>
 <text x="26.67" y="14.605" size="0.8128" layer="25" font="vector">(c)2016</text>
-<text x="1.905" y="1.27" size="0.762" layer="25" font="vector">OVERDRIVE/DIST</text>
-<text x="1.905" y="3.175" size="2.0828" layer="25" font="vector">JANUS</text>
+<text x="1.27" y="1.27" size="0.8636" layer="25" font="vector">OD+DISTORTION</text>
+<text x="1.27" y="2.54" size="2.2352" layer="25" font="vector">JANUS</text>
 </plain>
 <attributes>

Commit message: convert bitmap logos to polygons
Parts:
- added U$2: (no value), logos:RT0100
Changed lines of the file:
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@@
 <element name="R1" library="resistors" package="R0207/3" value="1M" x="26.67" y="3.81" rot="R180"/>
 <element name="9V" library="jacks" package="DC" value="DC_MONO" x="12.065" y="29.845" rot="MR0"/>
+<element name="U$2" library="logos" package="RT0100" value="" x="22.225" y="24.13" rot="R90"/>
 </elements>
 <signals>
