File: 1590a/janus_overdrive/janus.brd (EAGLE design)
At the start: 33 x 33 mm, 28 parts, among them IC1 LM741

Commit message: updated library + logos
Parts:
- removed U$2: (no value), logos:RT0100
- added U$1: (no value), logos:BF0100
Other:
- board text added: "http://bffx.us"
Changed lines of the file:
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@@
 <text x="1.27" y="1.27" size="0.8636" layer="25" font="vector">OD+DISTORTION</text>
 <text x="1.27" y="2.54" size="2.2352" layer="25" font="vector">JANUS</text>
+<text x="12.065" y="5.08" size="0.8128" layer="25" font="vector">http://bffx.us</text>
 </plain>
 <attributes>
@@
 <element name="R1" library="resistors" package="R0207/3" value="1M" x="26.67" y="3.81" rot="R180"/>
 <element name="9V" library="jacks" package="DC" value="DC_MONO" x="12.065" y="29.845" rot="MR0"/>
-<element name="U$2" library="logos" package="RT0100" value="" x="22.225" y="24.13" rot="R90"/>
+<element name="U$1" library="logos" package="BF0100" value="" x="22.225" y="23.495"/>
 </elements>
 <signals>
