File: 1590a/janus_overdrive/janus.sch (EAGLE design)
At the start: 28 parts, among them IC1 LM741

Commit message: finished chorus and tremolo baords; other tweaks & polish
Parts:
- removed PAD1, PAD2: PADSQR, supply pins:PADSQR
- removed PAD4: PADRND, supply pins:PADRND
- added 9V: DC_MONO, jacks:DC_MONO
- added IN: PADSQR, supply pins:PADSQR
- C1, C3, C5: device capacitors-film:CER/FILMBOX.1 -> capacitors-film:CER/FILM2
- D1: device diodes:DO41.2 -> diodes:DO41.3
- renumbered PAD3 to GND, PAD5 to OUT
Connections:
- removed net +9V: D1.A, PAD1.P$1
- new net N$11: 9V.TIP, D1.A
- net GND: now also 9V.SLEEVE; no longer PAD4.P$1
- net IN: now also IN.P$1; no longer PAD2.P$1
Other:
- note added: "JANUS"
- note added: "OVERDRIVE / DISTORTION mashup of the dan armstrong blue clipper, mxr dist+, dod 250, and mxr microamp (c)2016 burr settles"
- note removed: "JANUS DRIVE"
- note removed: "OVERDRIVE / DISTORTION mashup of the dan armstrong blue clipper, mxr dist+, dod 250, and mxr microamp (c) 2016 burr settles"
- moved on the sheet: D1
Changed lines of the file:
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@@
 <drawing>
 <settings>
-<setting alwaysvectorfont="no"/>
+<setting alwaysvectorfont="yes"/>
 <setting verticaltext="up"/>
 </settings>
@@
 <part name="R2" library="resistors" deviceset="R_" device=".3B" value="22k"/>
 <part name="R6" library="resistors" deviceset="R_" device=".3B" value="470k"/>
-<part name="C5" library="capacitors-film" deviceset="CER/FILM" device="BOX.1" value="47n"/>
+<part name="C5" library="capacitors-film" deviceset="CER/FILM" device="2" value="47n"/>
 <part name="R4" library="resistors" deviceset="R_" device=".3B" value="4k7"/>
 <part name="IC1" library="integrated circuits" deviceset="SINGLE" device="TH" value="LM741"/>
@@
 <part name="D2" library="diodes" deviceset="DO35" device=".2"/>
 <part name="D3" library="diodes" deviceset="DO35" device=".2"/>
-<part name="C3" library="capacitors-film" deviceset="CER/FILM" device="BOX.1" value="10n"/>
-<part name="C1" library="capacitors-film" deviceset="CER/FILM" device="BOX.1" value="2n2"/>
+<part name="C3" library="capacitors-film" deviceset="CER/FILM" device="2" value="10n"/>
+<part name="C1" library="capacitors-film" deviceset="CER/FILM" device="2" value="2n2"/>
 <part name="C4" library="capacitors-elec" deviceset="050" device="1" value="10u"/>
 <part name="VOLUME" library="potentiometers" deviceset="POTS" device="SMALL_PADS" value="100kA"/>
-<part name="V1" library="gm-supply" deviceset="+9V" device=""/>
 <part name="GND1" library="gm-supply" deviceset="GND" device=""/>
 <part name="GND8" library="gm-supply" deviceset="GND" device=""/>
@@
 <part name="GND5" library="gm-supply" deviceset="GND" device=""/>
 <part name="GND6" library="gm-supply" deviceset="GND" device=""/>
-<part name="IN1" library="gm-supply" deviceset="IN" device=""/>
-<part name="OUT1" library="gm-supply" deviceset="OUT" device=""/>
 <part name="GND7" library="gm-supply" deviceset="GND" device=""/>
-<part name="PAD1" library="supply pins" deviceset="PAD" device="SQR"/>
-<part name="PAD2" library="supply pins" deviceset="PAD" device="SQR"/>
-<part name="PAD5" library="supply pins" deviceset="PAD" device="SQR"/>
-<part name="PAD3" library="supply pins" deviceset="PAD" device="RND"/>
-<part name="PAD4" library="supply pins" deviceset="PAD" device="RND"/>
+<part name="IN" library="supply pins" deviceset="PAD" device="SQR"/>
+<part name="OUT" library="supply pins" deviceset="PAD" device="SQR"/>
+<part name="GND" library="supply pins" deviceset="PAD" device="RND"/>
 <part name="DRIVE" library="potentiometers" deviceset="POTS" device="SMALL_PADS" value="500kC"/>
 <part name="CLIP" library="switches" deviceset="SPDT" device="PADS"/>
@@
 <part name="GND10" library="gm-supply" deviceset="GND" device=""/>
 <part name="GND11" library="gm-supply" deviceset="GND" device=""/>
-<part name="D1" library="diodes" deviceset="DO41" device=".2" value="1N5817"/>
+<part name="D1" library="diodes" deviceset="DO41" device=".3" value="1N5817"/>
 <part name="C2" library="capacitors-elec" deviceset="050" device="1" value="47u"/>
 <part name="GND3" library="gm-supply" deviceset="GND" device=""/>
 <part name="R1" library="resistors" deviceset="R_" device=".3B" value="1M"/>
+<part name="9V" library="jacks" deviceset="DC_MONO" device=""/>
+<part name="GND13" library="gm-supply" deviceset="GND" device=""/>
 </parts>
 <sheets>
 <sheet>
 <plain>
-<text x="78.74" y="73.66" size="6.4516" layer="97">JANUS DRIVE</text>
+<text x="78.74" y="73.66" size="6.4516" layer="97">JANUS</text>
 <text x="78.74" y="60.96" size="1.9304" layer="97">OVERDRIVE / DISTORTION
 mashup of the dan armstrong blue clipper,
 mxr dist+, dod 250, and mxr microamp
-(c) 2016 burr settles</text>
+(c)2016 burr settles</text>
 </plain>
 <instances>
@@
 <instance part="C4" gate="1" x="50.8" y="58.42" rot="MR270"/>
 <instance part="VOLUME" gate="G$1" x="134.62" y="25.4"/>
-<instance part="V1" gate="+9V" x="7.62" y="81.28" rot="R90"/>
 <instance part="GND1" gate="GND" x="15.24" y="7.62"/>
 <instance part="GND8" gate="GND" x="99.06" y="7.62"/>
@@
 <instance part="GND5" gate="GND" x="40.64" y="50.8"/>
 <instance part="GND6" gate="GND" x="50.8" y="50.8"/>
-<instance part="IN1" gate="G$1" x="7.62" y="38.1"/>
-<instance part="OUT1" gate="G$1" x="147.32" y="25.4"/>
 <instance part="GND7" gate="GND" x="68.58" y="25.4"/>
-<instance part="PAD1" gate="G$1" x="10.16" y="81.28"/>
-<instance part="PAD2" gate="G$1" x="10.16" y="38.1"/>
-<instance part="PAD5" gate="G$1" x="144.78" y="25.4"/>
-<instance part="PAD3" gate="G$1" x="15.24" y="10.16" rot="R90"/>
-<instance part="PAD4" gate="G$1" x="134.62" y="10.16" rot="R90"/>
+<instance part="IN" gate="G$1" x="7.62" y="38.1"/>
+<instance part="OUT" gate="G$1" x="144.78" y="25.4"/>
+<instance part="GND" gate="G$1" x="15.24" y="10.16" rot="R90"/>
 <instance part="DRIVE" gate="G$1" x="35.56" y="20.32"/>
 <instance part="CLIP" gate="1" x="111.76" y="27.94" rot="R180"/>
@@
 <instance part="GND10" gate="GND" x="114.3" y="7.62"/>
 <instance part="GND11" gate="GND" x="119.38" y="7.62"/>
-<instance part="D1" gate="G$1" x="17.78" y="81.28"/>
+<instance part="D1" gate="G$1" x="20.32" y="81.28"/>
 <instance part="C2" gate="1" x="30.48" y="73.66" rot="MR270"/>
 <instance part="GND3" gate="GND" x="30.48" y="66.04"/>
 <instance part="R1" gate="G$1" x="15.24" y="27.94" rot="R90"/>
+<instance part="9V" gate="DC" x="5.08" y="78.74"/>
+<instance part="GND13" gate="GND" x="10.16" y="73.66"/>
 </instances>
 <busses>
@@
 <segment>
 <pinref part="GND1" gate="GND" pin="GND"/>
-<pinref part="PAD3" gate="G$1" pin="P$1"/>
+<pinref part="GND" gate="G$1" pin="P$1"/>
 <wire x1="15.24" y1="10.16" x2="15.24" y2="22.86" width="0.1524" layer="91"/>
 <junction x="15.24" y="10.16"/>
@@
 <pinref part="GND12" gate="GND" pin="GND"/>
 <pinref part="VOLUME" gate="G$1" pin="1"/>
-<pinref part="PAD4" gate="G$1" pin="P$1"/>
 <wire x1="134.62" y1="10.16" x2="134.62" y2="19.05" width="0.1524" layer="91"/>
-<junction x="134.62" y="10.16"/>
 </segment>
 <segment>
@@
 <pinref part="GND3" gate="GND" pin="GND"/>
 </segment>
-</net>
-<net name="IN" class="0">
-<segment>
-<pinref part="IN1" gate="G$1" pin="IN"/>
-<pinref part="C3" gate="G$1" pin="2"/>
-<wire x1="10.16" y1="38.1" x2="15.24" y2="38.1" width="0.1524" layer="91"/>
-<wire x1="15.24" y1="38.1" x2="25.4" y2="38.1" width="0.1524" layer="91"/>
-<junction x="15.24" y="38.1"/>
-<pinref part="PAD2" gate="G$1" pin="P$1"/>
-<junction x="10.16" y="38.1"/>
-<pinref part="R1" gate="G$1" pin="2"/>
-<wire x1="25.4" y1="38.1" x2="39.37" y2="38.1" width="0.1524" layer="91"/>
-<wire x1="15.24" y1="33.02" x2="15.24" y2="38.1" width="0.1524" layer="91"/>
-<junction x="25.4" y="38.1"/>
-<pinref part="C1" gate="G$1" pin="2"/>
-<wire x1="25.4" y1="31.75" x2="25.4" y2="38.1" width="0.1524" layer="91"/>
-</segment>
-</net>
-<net name="OUT" class="0">
-<segment>
-<pinref part="OUT1" gate="G$1" pin="OUT"/>
-<pinref part="VOLUME" gate="G$1" pin="2"/>
-<pinref part="PAD5" gate="G$1" pin="P$1"/>
-<wire x1="144.78" y1="25.4" x2="139.7" y2="25.4" width="0.1524" layer="91"/>
-<junction x="144.78" y="25.4"/>
-</segment>
-</net>
-<net name="+9V" class="0">
-<segment>
-<pinref part="D1" gate="G$1" pin="A"/>
-<wire x1="10.16" y1="81.28" x2="12.7" y2="81.28" width="0.1524" layer="91"/>
-<pinref part="PAD1" gate="G$1" pin="P$1"/>
-<junction x="10.16" y="81.28"/>
-<pinref part="V1" gate="+9V" pin="+9V"/>
+<segment>
+<pinref part="9V" gate="DC" pin="SLEEVE"/>
+<pinref part="GND13" gate="GND" pin="GND"/>
 </segment>
 </net>
@@
 <segment>
 <pinref part="IC1" gate="A" pin="V+"/>
-<wire x1="20.32" y1="81.28" x2="30.48" y2="81.28" width="0.1524" layer="91"/>
+<wire x1="22.86" y1="81.28" x2="30.48" y2="81.28" width="0.1524" layer="91"/>
 <wire x1="30.48" y1="81.28" x2="40.64" y2="81.28" width="0.1524" layer="91"/>
 <wire x1="40.64" y1="81.28" x2="68.58" y2="81.28" width="0.1524" layer="91"/>
@@
 </segment>
 </net>
+<net name="N$11" class="0">
+<segment>
+<pinref part="D1" gate="G$1" pin="A"/>
+<wire x1="10.16" y1="81.28" x2="15.24" y2="81.28" width="0.1524" layer="91"/>
+<pinref part="9V" gate="DC" pin="TIP"/>
+</segment>
+</net>
+<net name="IN" class="0">
+<segment>
+<pinref part="C3" gate="G$1" pin="2"/>
+<wire x1="7.62" y1="38.1" x2="15.24" y2="38.1" width="0.1524" layer="91"/>
+<wire x1="15.24" y1="38.1" x2="25.4" y2="38.1" width="0.1524" layer="91"/>
+<junction x="15.24" y="38.1"/>
+<pinref part="IN" gate="G$1" pin="P$1"/>
+<pinref part="R1" gate="G$1" pin="2"/>
+<wire x1="25.4" y1="38.1" x2="39.37" y2="38.1" width="0.1524" layer="91"/>
+<wire x1="15.24" y1="33.02" x2="15.24" y2="38.1" width="0.1524" layer="91"/>
+<junction x="25.4" y="38.1"/>
+<pinref part="C1" gate="G$1" pin="2"/>
+<wire x1="25.4" y1="31.75" x2="25.4" y2="38.1" width="0.1524" layer="91"/>
+<label x="5.08" y="38.1" size="1.778" layer="95" rot="R180" xref="yes"/>
+<wire x1="5.08" y1="38.1" x2="7.62" y2="38.1" width="0.1524" layer="91"/>
+<junction x="7.62" y="38.1"/>
+</segment>
+</net>
+<net name="OUT" class="0">
+<segment>
+<pinref part="VOLUME" gate="G$1" pin="2"/>
+<pinref part="OUT" gate="G$1" pin="P$1"/>
+<wire x1="144.78" y1="25.4" x2="139.7" y2="25.4" width="0.1524" layer="91"/>
+<label x="147.32" y="25.4" size="1.778" layer="95" xref="yes"/>
+<wire x1="144.78" y1="25.4" x2="147.32" y2="25.4" width="0.1524" layer="91"/>
+<junction x="144.78" y="25.4"/>
+</segment>
+</net>

Commit message: added RT logo; converted some pots trimmers
Changed lines of the file:
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@@
 <part name="9V" library="jacks" deviceset="DC_MONO" device=""/>
 <part name="GND13" library="gm-supply" deviceset="GND" device=""/>
+<part name="U$1" library="logos" deviceset="REBELSTRUST" device=""/>
 </parts>
 <sheets>
 <sheet>
 <plain>
-<text x="78.74" y="73.66" size="6.4516" layer="97">JANUS</text>
-<text x="78.74" y="60.96" size="1.9304" layer="97">OVERDRIVE / DISTORTION
+<text x="76.2" y="78.74" size="6.4516" layer="97">JANUS</text>
+<text x="76.2" y="66.04" size="1.9304" layer="97">OVERDRIVE / DISTORTION
 mashup of the dan armstrong blue clipper,
 mxr dist+, dod 250, and mxr microamp
@@
 <instance part="9V" gate="DC" x="5.08" y="78.74"/>
 <instance part="GND13" gate="GND" x="10.16" y="73.66"/>
+<instance part="U$1" gate="G$1" x="76.2" y="53.34"/>
 </instances>
 <busses>

Commit message: little edits & cleanup
Other:
- note added: "OVERDRIVE + DISTORTION mashup of the dan armstrong blue clipper, mxr dist+, dod 250, and mxr microamp (c)2016 burr settles"
- note removed: "OVERDRIVE / DISTORTION mashup of the dan armstrong blue clipper, mxr dist+, dod 250, and mxr microamp (c)2016 burr settles"
- moved on the sheet: C6, R8
Changed lines of the file:
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@@
 <plain>
 <text x="76.2" y="78.74" size="6.4516" layer="97">JANUS</text>
-<text x="76.2" y="66.04" size="1.9304" layer="97">OVERDRIVE / DISTORTION
+<text x="76.2" y="66.04" size="1.9304" layer="97">OVERDRIVE + DISTORTION
 mashup of the dan armstrong blue clipper,
 mxr dist+, dod 250, and mxr microamp
@@
 <instance part="IC1" gate="A" x="71.12" y="35.56"/>
 <instance part="R7" gate="G$1" x="76.2" y="17.78"/>
-<instance part="C6" gate="1" x="86.36" y="35.56"/>
-<instance part="R8" gate="G$1" x="99.06" y="35.56"/>
+<instance part="C6" gate="1" x="88.9" y="35.56"/>
+<instance part="R8" gate="G$1" x="101.6" y="35.56"/>
 <instance part="D2" gate="G$1" x="99.06" y="15.24" rot="R90"/>
 <instance part="D3" gate="G$1" x="104.14" y="12.7" rot="R270"/>
@@
 <wire x1="78.74" y1="35.56" x2="81.28" y2="35.56" width="0.1524" layer="91"/>
 <pinref part="R7" gate="G$1" pin="2"/>
-<wire x1="81.28" y1="35.56" x2="83.82" y2="35.56" width="0.1524" layer="91"/>
+<wire x1="81.28" y1="35.56" x2="86.36" y2="35.56" width="0.1524" layer="91"/>
 <junction x="81.28" y="35.56"/>
 <wire x1="81.28" y1="17.78" x2="81.28" y2="35.56" width="0.1524" layer="91"/>
@@
 <pinref part="C6" gate="1" pin="-"/>
 <pinref part="R8" gate="G$1" pin="1"/>
-<wire x1="93.98" y1="35.56" x2="91.44" y2="35.56" width="0.1524" layer="91"/>
+<wire x1="96.52" y1="35.56" x2="93.98" y2="35.56" width="0.1524" layer="91"/>
 </segment>
 </net>
@@
 <pinref part="VOLUME" gate="G$1" pin="3"/>
 <pinref part="R8" gate="G$1" pin="2"/>
-<wire x1="104.14" y1="35.56" x2="109.22" y2="35.56" width="0.1524" layer="91"/>
+<wire x1="106.68" y1="35.56" x2="109.22" y2="35.56" width="0.1524" layer="91"/>
 <pinref part="CLIP" gate="1" pin="P"/>
 <wire x1="109.22" y1="35.56" x2="134.62" y2="35.56" width="0.1524" layer="91"/>

Commit message: updated library + logos
Other:
- note added: "OVERDRIVE + DISTORTION mashup of the dan armstrong blue clipper, mxr dist+, dod 250, and mxr microamp (c)2016 burr settles - http://bffx.us"
- note removed: "OVERDRIVE + DISTORTION mashup of the dan armstrong blue clipper, mxr dist+, dod 250, and mxr microamp (c)2016 burr settles"
Changed lines of the file:
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@@
 <part name="9V" library="jacks" deviceset="DC_MONO" device=""/>
 <part name="GND13" library="gm-supply" deviceset="GND" device=""/>
-<part name="U$1" library="logos" deviceset="REBELSTRUST" device=""/>
+<part name="BF1" library="logos" deviceset="BULLFINCH" device=""/>
 </parts>
 <sheets>
@@
 mashup of the dan armstrong blue clipper,
 mxr dist+, dod 250, and mxr microamp
-(c)2016 burr settles</text>
+(c)2016 burr settles - http://bffx.us</text>
 </plain>
 <instances>
@@
 <instance part="9V" gate="DC" x="5.08" y="78.74"/>
 <instance part="GND13" gate="GND" x="10.16" y="73.66"/>
-<instance part="U$1" gate="G$1" x="76.2" y="53.34"/>
+<instance part="BF1" gate="G$1" x="81.28" y="58.42"/>
 </instances>
 <busses>
