File: 1590a/siren_chorus/siren.brd (EAGLE design)
At the start: 33 x 52.7 mm, 52 parts, among them IC1 NE5532, Q1 2N5457

Commit message: finished chorus and tremolo baords; other tweaks & polish
Parts:
- added PAD1: PAD, supply pins:UNLABELED
- moved GND 3.18 mm to (29.2, 2.54)
- moved OUT 3.18 mm to (26.0, 2.54)
- moved R12 1.42 mm to (10.8, 40.6)
- moved PAD2 1.27 mm to (8.89, 2.54)
- moved C13 0.64 mm to (12.7, 24.1)
- moved R14 0.64 mm to (12.7, 21.6)
- moved C3 0.63 mm to (12.7, 11.4)
- moved R8 0.63 mm to (12.7, 14.0)
- moved 9V 0.63 mm to (12.7, 50.8)
- moved C1 0.63 mm to (27.9, 46.4)
- moved C10 0.63 mm to (12.7, 16.5)
- moved C2 0.63 mm to (3.81, 43.2)
- moved D1 0.63 mm to (6.35, 47.6)
- moved DEPTH 0.63 mm to (5.08, 50.8)
- moved IC1 0.63 mm to (18.4, 41.9)
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- renumbered LED to L+
Connections:
- net VC: now also PAD1.P$1
Routing:
- net VC: track 0.00 -> 89.0 mm
- net LED: track 0.00 -> 63.0 mm
- net N$13: track 0.00 -> 36.2 mm
- net N$28: track 0.00 -> 29.3 mm
- net N$19: track 0.00 -> 27.7 mm
- net N$31: track 0.00 -> 25.0 mm
- net N$14: track 0.00 -> 20.4 mm
- net N$24: track 0.00 -> 18.5 mm
- net N$21: track 0.00 -> 17.7 mm
- net N$5: track 0.00 -> 12.0 mm
- net N$25: track 0.00 -> 11.9 mm
- net N$18: track 0.00 -> 10.2 mm
- net N$3: track 0.00 -> 10.1 mm
- net N$26: track 0.00 -> 9.99 mm
- net N$20: track 0.00 -> 9.83 mm
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Other:
- board size 33 x 52.7 mm -> 33 x 53.3 mm
- board text added: "(c)2016"
- board text added: "SIREN CHORUS"
- board text added: "burr settles"

Commit message: prettified schematics a bit
Other:
- board text added: "6vTEST"
Changed lines of the file:
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@@
 <grid distance="25" unitdist="mil" unit="mil" style="lines" multiple="4" display="no" altdistance="0.025" altunitdist="inch" altunit="inch"/>
 <layers>
-<layer number="1" name="Top" color="4" fill="1" visible="yes" active="yes"/>
-<layer number="16" name="Bottom" color="1" fill="1" visible="yes" active="yes"/>
+<layer number="1" name="Top" color="4" fill="1" visible="no" active="yes"/>
+<layer number="16" name="Bottom" color="1" fill="1" visible="no" active="yes"/>
 <layer number="17" name="Pads" color="2" fill="1" visible="yes" active="yes"/>
 <layer number="18" name="Vias" color="2" fill="1" visible="yes" active="yes"/>
@@
 <wire x1="0" y1="53.34" x2="0" y2="0" width="0" layer="20"/>
 <text x="6.985" y="34.925" size="1.778" layer="25">SIREN CHORUS</text>
-<text x="9.525" y="4.445" size="0.8128" layer="25" rot="R90">(c)2016</text>
+<text x="17.145" y="52.07" size="0.8128" layer="25">(c)2016</text>
 <text x="24.13" y="48.26" size="0.8128" layer="25">burr settles</text>
+<text x="8.89" y="6.35" size="0.8128" layer="25" rot="R90" align="center">6vTEST</text>
 </plain>
 <attributes>
@@
 <contactref element="C12" pad="-"/>
 <contactref element="C9" pad="2"/>
+<contactref element="GND" pad="1"/>
+<contactref element="9V" pad="S"/>
 <contactref element="IC2" pad="4"/>
 <contactref element="IC2" pad="3"/>
 <contactref element="C14" pad="2"/>
 <contactref element="C17" pad="2"/>
-<contactref element="GND" pad="1"/>
-<contactref element="9V" pad="S"/>
 </signal>
 <signal name="VC">
@@
 <wire x1="17.78" y1="9.525" x2="18.415" y2="10.16" width="0.254" layer="1"/>
 </signal>
-<signal name="N$14">
-<contactref element="IC2" pad="13"/>
-<contactref element="C13" pad="1"/>
-<contactref element="R10" pad="2"/>
-<contactref element="R17" pad="1"/>
-<contactref element="R15" pad="2"/>
-<wire x1="2.54" y1="22.86" x2="5.08" y2="22.86" width="0.254" layer="16"/>
-<wire x1="5.08" y1="22.86" x2="7.62" y2="25.4" width="0.254" layer="16"/>
-<wire x1="7.62" y1="25.4" x2="7.62" y2="27.94" width="0.254" layer="16"/>
-<wire x1="15.24" y1="24.13" x2="16.51" y2="24.13" width="0.254" layer="16"/>
-<wire x1="16.51" y1="24.13" x2="17.78" y2="22.86" width="0.254" layer="16"/>
-<wire x1="15.24" y1="24.13" x2="13.97" y2="24.13" width="0.254" layer="16"/>
-<wire x1="13.97" y1="24.13" x2="12.065" y2="26.035" width="0.254" layer="16"/>
-<wire x1="12.065" y1="26.035" x2="8.255" y2="26.035" width="0.254" layer="16"/>
-<wire x1="8.255" y1="26.035" x2="7.62" y2="25.4" width="0.254" layer="16"/>
-</signal>
 <signal name="N$15">
 <contactref element="R14" pad="2"/>
@@
 <wire x1="11.43" y1="48.895" x2="10.16" y2="47.625" width="0.6096" layer="1"/>
 </signal>
+<signal name="N$1">
+<contactref element="IC2" pad="13"/>
+<contactref element="C13" pad="1"/>
+<contactref element="R10" pad="2"/>
+<contactref element="R17" pad="1"/>
+<contactref element="R15" pad="2"/>
+<wire x1="2.54" y1="22.86" x2="5.08" y2="22.86" width="0.254" layer="16"/>
+<wire x1="5.08" y1="22.86" x2="7.62" y2="25.4" width="0.254" layer="16"/>
+<wire x1="7.62" y1="25.4" x2="7.62" y2="27.94" width="0.254" layer="16"/>
+<wire x1="15.24" y1="24.13" x2="16.51" y2="24.13" width="0.254" layer="16"/>
+<wire x1="16.51" y1="24.13" x2="17.78" y2="22.86" width="0.254" layer="16"/>
+<wire x1="15.24" y1="24.13" x2="13.97" y2="24.13" width="0.254" layer="16"/>
+<wire x1="13.97" y1="24.13" x2="12.065" y2="26.035" width="0.254" layer="16"/>
+<wire x1="12.065" y1="26.035" x2="8.255" y2="26.035" width="0.254" layer="16"/>
+<wire x1="8.255" y1="26.035" x2="7.62" y2="25.4" width="0.254" layer="16"/>
+</signal>
 </signals>

Commit message: added RT logo; converted some pots trimmers
Parts:
- added U$1: (no value), logos:RT150
- DEPTH: device potentiometers:PADS_SMALL -> potentiometers:2262_TRIM
- moved C4 4.84 mm to (8.26, 39.4)
- moved C2 3.42 mm to (2.54, 40.0), turned to 270 degrees
- moved D1 3.17 mm to (6.35, 44.5)
- moved R12 1.90 mm to (12.7, 40.6)
- moved IC1 0.64 mm to (19.1, 41.9)
- moved DEPTH 0.63 mm to (5.08, 50.2), turned to 180 degrees
Routing:
- net LED: track 63.0 -> 71.5 mm
- net N$28: track 29.3 -> 23.3 mm
- net +9V: track 3.70 -> 6.88 mm
- net N$31: track 25.0 -> 22.3 mm
- net N$19: track 27.7 -> 29.0 mm
- net N$26: track 9.99 -> 11.1 mm
- net VC: track 89.0 -> 88.1 mm
Other:
- board text added: "<SIREN//CHORUS>"
- board text removed: "SIREN CHORUS"

Commit message: convert bitmap logos to polygons
Parts:
- removed U$1: (no value), logos:RT150
- added U$3: (no value), logos:RT0150
Changed lines of the file:
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@@
 <element name="L+" library="supply pins" package="SQUARE" value="PADSQR" x="22.86" y="2.54"/>
 <element name="PAD1" library="supply pins" package="UNLABELED" value="PAD" x="24.765" y="10.795"/>
-<element name="U$1" library="logos" package="RT150" value="" x="10.16" y="45.72"/>
+<element name="U$3" library="logos" package="RT0150" value="" x="12.065" y="47.371"/>
 </elements>
 <signals>
