File: 1590a/siren_chorus/siren.brd (EAGLE design)
At the start: 33 x 53.3 mm, 54 parts, among them IC1 NE5532, Q1 2N5457

Commit message: updated library + logos
Parts:
- removed U$3: (no value), logos:RT0150
- added U$1: (no value), logos:BF0150
Other:
- board text added: "http://bffx.us"
Changed lines of the file:
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@@
 <text x="8.89" y="6.35" size="0.8128" layer="25" rot="R90" align="center">6vTEST</text>
 <text x="1.905" y="34.798" size="1.778" layer="25">&lt;SIREN//CHORUS&gt;</text>
+<text x="1.27" y="43.18" size="0.8128" layer="25" rot="R90">http://bffx.us</text>
 </plain>
 <attributes>
@@
 <element name="L+" library="supply pins" package="SQUARE" value="PADSQR" x="22.86" y="2.54"/>
 <element name="PAD1" library="supply pins" package="UNLABELED" value="PAD" x="24.765" y="10.795"/>
-<element name="U$3" library="logos" package="RT0150" value="" x="12.065" y="47.371"/>
+<element name="U$1" library="logos" package="BF0150" value="" x="11.43" y="46.99" rot="R90"/>
 </elements>
 <signals>
