File: 1590a/siren_chorus/siren.sch (EAGLE design)
At the start: 53 parts, among them IC1 NE5532, Q1 2N5457

Commit message: updated library + logos
Other:
- note added: "PT2399 CHORUS based on the madbeanpedals glam (c)2016 burr settles - http://bffx.us"
- note removed: "PT2399 CHORUS based on the madbeanpedals glam (c)2016 burr settles"
Changed lines of the file:
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@@
 <part name="PAD1" library="supply pins" deviceset="PAD" device=""/>
 <part name="GND8" library="supply pins" deviceset="GND" device=""/>
-<part name="U$1" library="logos" deviceset="REBELSTRUST" device=""/>
+<part name="BF1" library="logos" deviceset="BULLFINCH" device=""/>
 </parts>
 <sheets>
@@
 <text x="5.08" y="124.46" size="1.9304" layer="97">PT2399 CHORUS
 based on the madbeanpedals glam
-(c)2016 burr settles</text>
+(c)2016 burr settles - http://bffx.us</text>
 <text x="5.08" y="134.62" size="6.4516" layer="97">SIREN</text>
 </plain>
@@
 <instance part="PAD1" gate="G$1" x="81.28" y="78.74"/>
 <instance part="GND8" gate="GND" x="203.2" y="48.26"/>
-<instance part="U$1" gate="G$1" x="5.08" y="111.76"/>
+<instance part="BF1" gate="G$1" x="38.1" y="137.16"/>
 </instances>
 <busses>
