File: 1590b/chimera_chorus/chimera.sch (EAGLE design)
At the start: 42 parts, among them IC1 TL072, IC2 TL072, IC3 MN3007, IC4 CD4046

Commit message: prettified schematics a bit
Parts:
- removed PAD1, PAD3: PADSQR, supply pins:PADSQR
- removed PAD5: PADRND, supply pins:PADRND
- added IN: PADSQR, supply pins:PADSQR
- added U$1: DC_MONO, jacks:DC_MONO
- C1: value 470uF -> 470u
- C2, C5, C8, C9: device capacitors-film:CER/FILMBOX.1 -> capacitors-film:CER/FILM2
- C3: value 10uF -> 10u
- C6: device capacitors-film:CER/FILMBOX.2 -> capacitors-film:CER/FILM2
- renumbered PAD2 to OUT, PAD4 to GND
Connections:
- removed net +9V: D1.A, PAD3.P$1
- removed net N$25: R17.1, VIBE_B.1
- removed net VA: C1.+, D1.C, IC1_PWR.V+, IC2_PWR.V+, IC3.1, IC4.14, IC4.16, R11.2, R4.2
- new net N$26: C3.+, IC2_A.-IN, R2.1, R3.2, R4.2, R5.1, R7.1
- new net N$29: D1.A, U$1.TIP
- new net VC: C1.+, D1.C, IC1_PWR.V+, IC2_PWR.V+, IC3.1, IC4.14, IC4.16, R11.1, R4.1
- net GND: now also U$1.SLEEVE; no longer PAD5.P$1
- net IN: now also IN.P$1; no longer PAD1.P$1
- net N$10: now also DEPTH.3, IC2_B.OUT, R9.2; no longer IC2_B.+IN, R10.2
- net N$16: now also R11.2, R12.1; no longer R11.1, R12.2
- net N$17: now also R16.2; no longer R16.1
- net N$18: now also R12.2, R15.1; no longer R12.1, R15.2
- net N$19: now also R15.2, R16.1; no longer R15.1, R16.2
- net N$23: now also VIBE_B.1; no longer VIBE_A.1
- net N$5: now also IC2_B.+IN, R10.2; no longer DEPTH.3, IC2_B.OUT, R9.1
- net N$6: now also R17.1, VIBE_A.1; no longer C3.+, IC2_A.-IN, R2.1, R3.2, R4.1, R5.1, R7.1
- net N$7: now also R8.1, R9.1; no longer R8.2, R9.2
- net N$8: now also R8.2; no longer R8.1
Other:
- moved on the sheet: C1, C2, C3, C4, C5, C6, C7, C8, C9, D1, DEPTH, IC1_B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

Commit message: convert bitmap logos to polygons
Changed lines of the file:
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@@
 <setting verticaltext="up"/>
 </settings>
-<grid distance="0.05" unitdist="inch" unit="inch" style="lines" multiple="2" display="no" altdistance="0.01" altunitdist="inch" altunit="inch"/>
+<grid distance="0.1" unitdist="inch" unit="inch" style="lines" multiple="1" display="no" altdistance="0.01" altunitdist="inch" altunit="inch"/>
 <layers>
 <layer number="1" name="Top" color="4" fill="1" visible="no" active="no"/>
@@
 <net name="IN" class="0">
 <segment>
-<wire x1="-12.7" y1="78.74" x2="-10.16" y2="78.74" width="0.1524" layer="91"/>
+<wire x1="-17.78" y1="78.74" x2="-10.16" y2="78.74" width="0.1524" layer="91"/>
 <pinref part="R1" gate="G$1" pin="2"/>
 <wire x1="-10.16" y1="78.74" x2="-2.54" y2="78.74" width="0.1524" layer="91"/>
@@
 <pinref part="IN" gate="G$1" pin="P$1"/>
 <junction x="-10.16" y="78.74"/>
-<label x="-12.7" y="78.74" size="1.778" layer="95" rot="R180" xref="yes"/>
+<label x="-17.78" y="78.74" size="1.778" layer="95" rot="R180" xref="yes"/>
 </segment>
 </net>
@@
 <segment>
 <pinref part="C10" gate="G$1" pin="-"/>
-<wire x1="185.42" y1="81.28" x2="182.88" y2="81.28" width="0.1524" layer="91"/>
+<wire x1="190.5" y1="81.28" x2="182.88" y2="81.28" width="0.1524" layer="91"/>
 <pinref part="R18" gate="G$1" pin="2"/>
 <wire x1="182.88" y1="81.28" x2="180.34" y2="81.28" width="0.1524" layer="91"/>
@@
 <junction x="182.88" y="81.28"/>
 <pinref part="OUT" gate="G$1" pin="P$1"/>
-<label x="185.42" y="81.28" size="1.778" layer="95" xref="yes"/>
-</segment>
-</net>
+<label x="190.5" y="81.28" size="1.778" layer="95" xref="yes"/>
+</segment>
+</net>
