File: 1590a/cyclops_fuzz/cyclops.brd (EAGLE design)
At the start: 33 x 36.8 mm, 35 parts, among them IC1 CD4049

Commit message: updated library + logos
Parts:
- removed U$1: (no value), logos:RT0150
- added U$3: (no value), logos:BF0200
Other:
- board text added: "(c)2016 bullfinch fx"
- board text added: "http://bffx.us"
- board text removed: "(c)2016 burr settles"
Changed lines of the file:
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@@
 <setting verticaltext="up"/>
 </settings>
-<grid distance="0.025" unitdist="inch" unit="inch" style="lines" multiple="4" display="no" altdistance="0.025" altunitdist="inch" altunit="inch"/>
+<grid distance="0.0125" unitdist="inch" unit="inch" style="lines" multiple="4" display="no" altdistance="0.025" altunitdist="inch" altunit="inch"/>
 <layers>
 <layer number="1" name="Top" color="4" fill="1" visible="yes" active="yes"/>
@@
 <text x="21.209" y="4.826" size="1.778" layer="25" rot="R90">CYCLOPS FUZZ</text>
 <text x="1.27" y="0.762" size="0.9652" layer="25">(c)2016
-burr settles</text>
+bullfinch fx</text>
+<text x="21.59" y="31.5595" size="0.9652" layer="25">http://bffx.us</text>
 </plain>
 <attributes>
@@
 <element name="GND" library="supply pins" package="ROUND" value="PADRND" x="15.875" y="2.54"/>
 <element name="D5" library="diodes" package="DO41-3" value="1N5417" x="13.335" y="34.29"/>
-<element name="U$1" library="logos" package="RT0150" value="" x="19.685" y="27.94" rot="R90"/>
+<element name="U$3" library="logos" package="BF0200" value="" x="19.05" y="29.845"/>
 </elements>
 <signals>
