File: 1590a/gaius_ringer/gaius.brd (EAGLE design)
At the start: 33 x 32.4 mm, 30 parts, among them Q1 2N5088, Q2 2N3906, Q3 2N5088

Commit message: add GAIUS documentation
Parts:
- NULL: value 25kB -> 100kB
Connections:
- net N$7: now also NULL.3; no longer NULL.1
Routing:
- net N$7: track 5.71 -> 8.94 mm
Changed lines of the file:
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@@
 <element name="D3" library="diodes" package="DO35-2" value="1N914" x="5.08" y="17.78" rot="R180"/>
 <element name="D1" library="diodes" package="DO41-3" value="1N5817" x="14.605" y="29.845"/>
-<element name="NULL" library="potentiometers" package="2262_TRIM" value="25kB" x="5.08" y="28.575" rot="R180"/>
+<element name="NULL" library="potentiometers" package="2262_TRIM" value="100kB" x="5.08" y="28.575" rot="R180"/>
 <element name="Q1" library="transistors" package="TO92-" value="2N5088" x="19.685" y="15.24" rot="R90"/>
 <element name="Q2" library="transistors" package="TO92-" value="2N3906" x="17.78" y="22.86" rot="R270"/>
@@
 <contactref element="R6" pad="1"/>
 <contactref element="Q2" pad="3"/>
-<wire x1="5.08" y1="26.035" x2="8.89" y2="26.035" width="0.254" layer="16"/>
 <wire x1="8.89" y1="26.035" x2="10.4775" y2="27.6225" width="0.254" layer="16"/>
 <wire x1="10.4775" y1="27.6225" x2="15.5575" y2="27.6225" width="0.254" layer="16"/>
@@
 <wire x1="19.3675" y1="25.4" x2="21.9075" y2="22.86" width="0.254" layer="16"/>
 <wire x1="21.9075" y1="22.86" x2="22.86" y2="22.86" width="0.254" layer="16"/>
+<wire x1="5.08" y1="26.035" x2="8.89" y2="26.035" width="0.254" layer="16"/>
 </signal>
 <signal name="N$6">
@@
 <wire x1="10.16" y1="12.7" x2="10.16" y2="10.16" width="0.254" layer="1"/>
 <wire x1="10.16" y1="10.16" x2="10.16" y2="7.62" width="0.254" layer="1"/>
-</signal>
-<signal name="N$7">
-<contactref element="C4" pad="1"/>
-<contactref element="NULL" pad="1"/>
-<wire x1="7.62" y1="28.575" x2="7.62" y2="22.86" width="0.254" layer="1"/>
 </signal>
 <signal name="N$8">
@@
 <wire x1="27.305" y1="29.845" x2="18.415" y2="29.845" width="0.6096" layer="1"/>
 </signal>
+<signal name="N$7">
+<contactref element="C4" pad="1"/>
+<contactref element="NULL" pad="3"/>
+<wire x1="7.62" y1="22.86" x2="5.715" y2="22.86" width="0.254" layer="1"/>
+<wire x1="5.715" y1="22.86" x2="2.54" y2="26.035" width="0.254" layer="1"/>
+<wire x1="2.54" y1="26.035" x2="2.54" y2="28.575" width="0.254" layer="1"/>
+</signal>
 </signals>

Commit message: updated library + logos
Parts:
- U$1: device logos:RT0150 -> logos:BF0150
- moved U$1 12.4 mm to (19.7, 7.62)
Other:
- board text added: "http://bffx.us"
Changed lines of the file:
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@@
 <text x="22.86" y="0.889" size="0.762" layer="25" font="vector">octavter +
 ring-modulator</text>
+<text x="9.525" y="27.178" size="0.8128" layer="25" font="vector">http://bffx.us</text>
 </plain>
 <attributes>
@@
 <element name="C5" library="capacitors-film" package="050X030_025_2" value="100n" x="13.335" y="10.16" rot="R90"/>
 <element name="9V" library="jacks" package="DC" value="DC_MONO" x="28.575" y="29.845" rot="MR0"/>
-<element name="U$1" library="logos" package="RT0150" value="" x="11.049" y="16.51"/>
+<element name="U$1" library="logos" package="BF0150" value="" x="19.685" y="7.62"/>
 </elements>
 <signals>
