File: 1590a/phrike_tremolo/phrike.brd (EAGLE design)
At the start: 33 x 41.9 mm, 38 parts, among them Q1 2N5457, Q2 2N3904, Q3 2N5457, Q4 2N5088

Commit message: add GAIUS documentation
Parts:
- R11: value 560k -> 1M
Changed lines of the file:
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@@
 <element name="R1" library="resistors" package="R0207/3" value="1M" x="2.54" y="5.715" rot="R90"/>
 <element name="R10" library="resistors" package="R0207/3" value="100k" x="6.35" y="30.48" rot="R180"/>
-<element name="R11" library="resistors" package="R0207/3" value="560k" x="6.35" y="33.02"/>
+<element name="R11" library="resistors" package="R0207/3" value="1M" x="6.35" y="33.02"/>
 <element name="R12" library="resistors" package="R0207/3" value="10k" x="14.605" y="20.32"/>
 <element name="R13" library="resistors" package="R0207/3" value="2M2" x="14.605" y="27.94" rot="R180"/>

Commit message: updated library + logos
Parts:
- removed U$2: (no value), logos:RT0150
- added U$1: (no value), logos:BF0150
Other:
- board text added: "http://bffx.us"
Changed lines of the file:
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@@
 <text x="18.415" y="8.89" size="1.1176" layer="25">TREMOLO</text>
 <text x="10.795" y="38.1" size="1.016" layer="25" rot="R90" align="bottom-center">(c)2016</text>
-<text x="21.082" y="23.495" size="1.0668" layer="25" rot="R90" align="bottom-center">burr settles</text>
+<text x="28.702" y="20.32" size="1.0668" layer="25" rot="R90" align="bottom-right">burr
+settles</text>
+<text x="21.082" y="23.495" size="1.0668" layer="25" rot="R90" align="bottom-center">http://bffx.us</text>
 </plain>
 <attributes>
@@
 <element name="C1" library="capacitors-elec" package="063_025" value="100u" x="18.415" y="33.655"/>
 <element name="9V" library="jacks" package="DC" value="DC_MONO" x="18.415" y="39.37" rot="MR0"/>
-<element name="U$2" library="logos" package="RT0150" value="" x="30.48" y="2.54"/>
+<element name="U$1" library="logos" package="BF0150" value="" x="30.48" y="3.175"/>
 </elements>
 <signals>
@@
 </board>
 </drawing>
+<compatibility>
+<note version="6.3" minversion="6.2.2" severity="warning">
+Since Version 6.2.2 text objects can contain more than one line,
+which will not be processed correctly with this version.
+</note>
+</compatibility>
 </eagle>
