File: 1590a/phrike_tremolo/phrike.sch (EAGLE design)
At the start: 37 parts, among them Q1 2N5457, Q2 2N3904, Q3 2N5457, Q4 2N5088

Commit message: finished chorus and tremolo baords; other tweaks & polish
Other:
- note added: "PHRIKE"
- note added: "TREMOLO based on the ea tremolo by anthony leo (electronics australia magazine, 1968) (c)2016 burr settles"
- note removed: "TREMOLO"
Changed lines of the file:
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@@
 <sheet>
 <plain>
-<text x="7.62" y="20.32" size="1.778" layer="97">TREMOLO</text>
+<text x="2.54" y="15.24" size="6.4516" layer="97">PHRIKE</text>
+<text x="2.54" y="2.54" size="1.9304" layer="97">TREMOLO
+based on the ea tremolo by anthony leo
+(electronics australia magazine, 1968)
+(c)2016 burr settles</text>
 </plain>
 <instances>
@@
 </schematic>
 </drawing>
+<compatibility>
+<note version="6.3" minversion="6.2.2" severity="warning">
+Since Version 6.2.2 text objects can contain more than one line,
+which will not be processed correctly with this version.
+</note>
+</compatibility>
 </eagle>

Commit message: added RT logo; converted some pots trimmers
Parts:
- DEPTH: device potentiometers:POTSSMALL_PADS -> potentiometers:POTSTRIM
Changed lines of the file:
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@@
 <part name="C4" library="capacitors-elec" deviceset="050" device="1" value="22u"/>
 <part name="Q3" library="transistors" deviceset="2N5457" device=""/>
-<part name="DEPTH" library="potentiometers" deviceset="POTS" device="SMALL_PADS" value="1MB"/>
+<part name="DEPTH" library="potentiometers" deviceset="POTS" device="TRIM" value="1MB"/>
 <part name="R10" library="resistors" deviceset="R_" device=".3B" value="100k"/>
 <part name="C6" library="capacitors-film" deviceset="CER/FILM" device="2" value="47n"/>
@@
 <part name="9V" library="jacks" deviceset="DC_MONO" device=""/>
 <part name="GND13" library="supply pins" deviceset="GND" device=""/>
+<part name="U$1" library="logos" deviceset="REBELSTRUST" device=""/>
 </parts>
 <sheets>
@@
 <instance part="9V" gate="DC" x="10.16" y="88.9"/>
 <instance part="GND13" gate="GND" x="17.78" y="83.82"/>
+<instance part="U$1" gate="G$1" x="2.54" y="25.4"/>
 </instances>
 <busses>

Commit message: add GAIUS documentation
Parts:
- R11: value 560k -> 1M
Changed lines of the file:
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@@
 <part name="GND11" library="supply pins" deviceset="GND" device=""/>
 <part name="GND12" library="supply pins" deviceset="GND" device=""/>
-<part name="R11" library="resistors" deviceset="R_" device=".3B" value="560k"/>
+<part name="R11" library="resistors" deviceset="R_" device=".3B" value="1M"/>
 <part name="GND9" library="supply pins" deviceset="GND" device=""/>
 <part name="GND1" library="supply pins" deviceset="GND" device=""/>

Commit message: updated library + logos
Changed lines of the file:
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@@
 <part name="9V" library="jacks" deviceset="DC_MONO" device=""/>
 <part name="GND13" library="supply pins" deviceset="GND" device=""/>
-<part name="U$1" library="logos" deviceset="REBELSTRUST" device=""/>
+<part name="BF1" library="logos" deviceset="BULLFINCH" device=""/>
 </parts>
 <sheets>
@@
 <instance part="9V" gate="DC" x="10.16" y="88.9"/>
 <instance part="GND13" gate="GND" x="17.78" y="83.82"/>
-<instance part="U$1" gate="G$1" x="2.54" y="25.4"/>
+<instance part="BF1" gate="G$1" x="7.62" y="30.48"/>
 </instances>
 <busses>
